File: RF-antenna/RF-VtoI.sch (EAGLE design)
At the start: 48 parts, among them CON1 UMC_CONNECTORREGULAR, CON2 UMC_CONNECTORREGULAR, CON3 UMC_CONNECTORREGULAR, CON4 UMC_CONNECTORREGULAR, CON5 UMC_CONNECTORREGULAR, CON6 UMC_CONNECTORREGULAR, U1 THS3091DDAR, U2 THS3091DDAR, U3 THS3091DDAR

Commit message: Starting full board layout
Got the VtoI converter designed and have started laying out the RF antennas.

DSB
Parts:
- removed C10, C15: 10nF, jqi_passives:C_MLCC_SMDCMLCC_0402
- removed C11, C12, C6, C7: 100nF, jqi_passives:C_MLCC_SMDCMLCC_0603
- removed C13, C14, C8, C9: 10uF, jqi_passives:C_MLCC_SMDCMLCC_1206
- removed CON3, CON4, CON5, CON6: UMC_CONNECTORREGULAR, qkdlab_alessandro:UMC_CONNECTORREGULAR
- removed JP2, JP3: (no value), pinhead:PINHD-1X3
- removed LG1, LG2: (no value), jqi_passives:L_FERRITE_SMD_1008
- removed LW1, LW2, LW3, LW4, LW5, LW6: LITZ_TERM, RFantenna:LITZ_TERM
- removed R2, R3: 49.9, jqi_passives:R_SMDR0402
- removed RF1, RF2: 866, jqi_passives:R_SMDR0603
- removed RG1, RG2: 95.3, jqi_passives:R_SMDR0402
- removed RS1, RS2: 10, jqi_passives:R_SMDR1206
- removed U1, U2: THS3091DDAR, opamp-jqi:THS3091DDAR
Connections:
- removed net D1_COIL: CON4.P$1, LW3.P1, LW4.P1, RF1.2, RS1.2, U1.OUT
- removed net D2_COIL: CON6.P$1, LW5.P1, LW6.P1, RF2.2, RS2.2, U2.OUT
- removed net N$10: LG1.2, RG1.2
- removed net N$11: RF2.1, RG2.1, U2.-IN
- removed net N$12: C15.2, R3.2, U2.+IN
- removed net N$13: C15.1, CON5.P$1
- removed net N$15: LG2.2, RG2.2
- removed net N$5: RF1.1, RG1.1, U1.-IN
- removed net N$7: C10.2, R2.2, U1.+IN
- removed net N$8: C10.1, CON3.P$1
- removed net R_COIL: CON1.P$1, LW1.P1, LW2.P1, RF.2, RS.2, U3.OUT
- new net N$2: CON1.P$1, RF.2, RS.2
- net +15V: no longer C12.1, C14.1, C7.1, C9.1, JP2.3, JP3.3, U1.V+, U2.V+
- net -15V: no longer C11.1, C13.1, C6.1, C8.1, JP2.1, JP3.1, U1.V-, U2.V-
- net GND: no longer C11.2, C12.2, C13.2, C14.2, C6.2, C7.2, C8.2, C9.2, CON3.P$2, CON3.P$3, CON4.P$2, CON4.P$3, CON5.P$2, CON5.P$3, CON6.P$2, CON6.P$3, JP2.2, JP3.2, LG1.1, LG2.1, R2.1, R3.1, RS1.1, RS2.1, U1.ON1, U1.ON2, U1.OPT, U2.ON1, U2.ON2, U2.OPT
