File: RF-antenna/RF-antenna.sch (EAGLE design)
At the start: 48 parts, among them CON1 UMC_CONNECTORREGULAR, CON2 UMC_CONNECTORREGULAR, CON3 UMC_CONNECTORREGULAR, CON4 UMC_CONNECTORREGULAR, CON5 UMC_CONNECTORREGULAR, CON6 UMC_CONNECTORREGULAR, U1 THS3091DDAR, U2 THS3091DDAR, U3 THS3091DDAR

Commit message: Test board ready
Pushing the prepared test board complete with 230 MHz and 6.8 GHz antennas for hyperfine control.

DSB
Parts:
- added C16: 3pF, jqi_passives:C_MLCC_SMDCMLCC_0402
- added C17: 0.3pF, jqi_passives:C_MLCC_SMDCMLCC_0402
- added X1, X2: SMA-V, connector-jqi:SMA-V
Connections:
- new net COIL6LI_N: C16.1, C16.2, C17.2, X2.2
- new net COIL6LI_P: C17.1, X2.1
- new net COIL87RB_GND: X1.2
- new net COIL87RB_IN: X1.1
Changed lines of the file:
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@@
 <class number="0" name="default" width="0" drill="0">
+</class>
+<class number="1" name="coupled" width="1.016" drill="0">
+<clearance class="1" value="0.381"/>
 </class>
 </classes>
@@
 <part name="LW5" library="RFantenna" deviceset="LITZ_TERM" device=""/>
 <part name="LW6" library="RFantenna" deviceset="LITZ_TERM" device=""/>
+<part name="X1" library="connector-jqi" deviceset="SMA" device="-V"/>
+<part name="X2" library="connector-jqi" deviceset="SMA" device="-V"/>
+<part name="FRAME1" library="frames" deviceset="FRAME_A_L" device=""/>
+<part name="C16" library="jqi_passives" deviceset="C_MLCC_SMD" device="CMLCC_0402" value="3pF">
+<attribute name="PARTNO" value="500R07S3R0BV4T"/>
+</part>
+<part name="C17" library="jqi_passives" deviceset="C_MLCC_SMD" device="CMLCC_0402" value="0.3pF">
+<attribute name="PARTNO" value="500R07S0R3AV4T"/>
+</part>
 </parts>
 <sheets>
@@
 </segment>
 </net>
+</nets>
+</sheet>
+<sheet>
+<plain>
+</plain>
+<instances>
+<instance part="X1" gate="G$1" x="35.56" y="67.31"/>
+<instance part="X2" gate="G$1" x="34.29" y="26.67"/>
+<instance part="FRAME1" gate="G$1" x="0" y="0"/>
+<instance part="FRAME1" gate="G$2" x="172.72" y="0"/>
+<instance part="C16" gate="G$1" x="59.69" y="26.67">
+<attribute name="PARTNO" x="59.69" y="26.67" size="1.778" layer="96" rot="R270" display="off"/>
+</instance>
+<instance part="C17" gate="G$1" x="52.07" y="29.21" rot="R90">
+<attribute name="PARTNO" x="52.07" y="29.21" size="1.778" layer="96" display="off"/>
+</instance>
+</instances>
+<busses>
+</busses>
+<nets>
+<net name="COIL6LI_P" class="1">
+<segment>
+<pinref part="X2" gate="G$1" pin="1"/>
+<wire x1="36.83" y1="26.67" x2="36.83" y2="29.21" width="0.1524" layer="91"/>
+<label x="48.26" y="29.21" size="1.778" layer="95" rot="R90" xref="yes"/>
+<pinref part="C17" gate="G$1" pin="1"/>
+<wire x1="36.83" y1="29.21" x2="49.53" y2="29.21" width="0.1524" layer="91"/>
+</segment>
+</net>
+<net name="COIL6LI_N" class="1">
+<segment>
+<pinref part="X2" gate="G$1" pin="2"/>
+<wire x1="36.83" y1="21.59" x2="36.83" y2="24.13" width="0.1524" layer="91"/>
+<label x="48.26" y="21.59" size="1.778" layer="95" rot="R270" xref="yes"/>
+<pinref part="C16" gate="G$1" pin="2"/>
+<wire x1="59.69" y1="21.59" x2="36.83" y2="21.59" width="0.1524" layer="91"/>
+<wire x1="59.69" y1="21.59" x2="64.77" y2="21.59" width="0.1524" layer="91"/>
+<junction x="59.69" y="21.59"/>
+<wire x1="64.77" y1="21.59" x2="64.77" y2="29.21" width="0.1524" layer="91"/>
+<pinref part="C17" gate="G$1" pin="2"/>
+<pinref part="C16" gate="G$1" pin="1"/>
+<wire x1="57.15" y1="29.21" x2="59.69" y2="29.21" width="0.1524" layer="91"/>
+<wire x1="64.77" y1="29.21" x2="59.69" y2="29.21" width="0.1524" layer="91"/>
+<junction x="59.69" y="29.21"/>
+</segment>
+</net>
+<net name="COIL87RB_IN" class="0">
+<segment>
+<pinref part="X1" gate="G$1" pin="1"/>
+<wire x1="38.1" y1="67.31" x2="41.91" y2="67.31" width="0.1524" layer="91"/>
+<label x="41.91" y="67.31" size="1.778" layer="95" rot="R90" xref="yes"/>
+</segment>
+</net>
+<net name="COIL87RB_GND" class="0">
+<segment>
+<pinref part="X1" gate="G$1" pin="2"/>
+<wire x1="41.91" y1="64.77" x2="38.1" y2="64.77" width="0.1524" layer="91"/>
+<label x="41.91" y="64.77" size="1.778" layer="95" rot="R270" xref="yes"/>
+</segment>
+</net>

Commit message: Success
Got COMSOL to push, now updating with additional COMSOL and files for Macrofab.

DSB
Parts:
- added FID1, FID2, FID3, FID4, FID5, FID6, FID7, FID8: FIDUCIAL-1.0MM, fiducials-jqi:FIDUCIAL-1.0MM
- JP1, JP2, JP3, LG, LG1, LG2: value (none) -> DNP
- X1, X2: PARTNO (none) -> 5-1814832-1
Changed lines of the file:
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@@
 </part>
 <part name="GND5" library="supply1" library_urn="urn:adsk.eagle:library:371" deviceset="GND" device=""/>
-<part name="JP1" library="pinhead" deviceset="PINHD-1X3" device="">
+<part name="JP1" library="pinhead" deviceset="PINHD-1X3" device="" value="DNP">
 <attribute name="PARTNO" value="640456-3"/>
 </part>
@@
 <attribute name="PARTNO" value="1909763-1"/>
 </part>
-<part name="LG" library="jqi_passives" deviceset="L_FERRITE_SMD" device="_1008"/>
+<part name="LG" library="jqi_passives" deviceset="L_FERRITE_SMD" device="_1008" value="DNP"/>
 <part name="FRAME3" library="frames" deviceset="FRAME_A_L" device=""/>
 <part name="U1" library="opamp-jqi" deviceset="THS3091DDAR" device="">
@@
 </part>
 <part name="GND11" library="supply1" library_urn="urn:adsk.eagle:library:371" deviceset="GND" device=""/>
-<part name="JP2" library="pinhead" deviceset="PINHD-1X3" device="">
+<part name="JP2" library="pinhead" deviceset="PINHD-1X3" device="" value="DNP">
 <attribute name="PARTNO" value="640456-3"/>
 </part>
@@
 <attribute name="PARTNO" value="1909763-1"/>
 </part>
-<part name="LG1" library="jqi_passives" deviceset="L_FERRITE_SMD" device="_1008"/>
+<part name="LG1" library="jqi_passives" deviceset="L_FERRITE_SMD" device="_1008" value="DNP"/>
 <part name="FRAME4" library="frames" deviceset="FRAME_A_L" device=""/>
 <part name="U2" library="opamp-jqi" deviceset="THS3091DDAR" device="">
@@
 </part>
 <part name="GND17" library="supply1" library_urn="urn:adsk.eagle:library:371" deviceset="GND" device=""/>
-<part name="JP3" library="pinhead" deviceset="PINHD-1X3" device="">
+<part name="JP3" library="pinhead" deviceset="PINHD-1X3" device="" value="DNP">
 <attribute name="PARTNO" value="640456-3"/>
 </part>
@@
 <attribute name="PARTNO" value="1909763-1"/>
 </part>
-<part name="LG2" library="jqi_passives" deviceset="L_FERRITE_SMD" device="_1008"/>
+<part name="LG2" library="jqi_passives" deviceset="L_FERRITE_SMD" device="_1008" value="DNP"/>
 <part name="LW3" library="RFantenna" deviceset="LITZ_TERM" device=""/>
 <part name="LW4" library="RFantenna" deviceset="LITZ_TERM" device=""/>
 <part name="LW5" library="RFantenna" deviceset="LITZ_TERM" device=""/>
 <part name="LW6" library="RFantenna" deviceset="LITZ_TERM" device=""/>
-<part name="X1" library="connector-jqi" deviceset="SMA" device="-V"/>
-<part name="X2" library="connector-jqi" deviceset="SMA" device="-V"/>
+<part name="X1" library="connector-jqi" deviceset="SMA" device="-V">
+<attribute name="PARTNO" value="5-1814832-1"/>
+</part>
+<part name="X2" library="connector-jqi" deviceset="SMA" device="-V">
+<attribute name="PARTNO" value="5-1814832-1"/>
+</part>
 <part name="FRAME1" library="frames" deviceset="FRAME_A_L" device=""/>
 <part name="C16" library="jqi_passives" deviceset="C_MLCC_SMD" device="CMLCC_0402" value="3pF">
@@
 <attribute name="PARTNO" value="500R07S0R3AV4T"/>
 </part>
+<part name="FID1" library="fiducials-jqi" deviceset="FIDUCIAL" device="-1.0MM"/>
+<part name="FID2" library="fiducials-jqi" deviceset="FIDUCIAL" device="-1.0MM"/>
+<part name="FID3" library="fiducials-jqi" deviceset="FIDUCIAL" device="-1.0MM"/>
+<part name="FID4" library="fiducials-jqi" deviceset="FIDUCIAL" device="-1.0MM"/>
+<part name="FID5" library="fiducials-jqi" deviceset="FIDUCIAL" device="-1.0MM"/>
+<part name="FID6" library="fiducials-jqi" deviceset="FIDUCIAL" device="-1.0MM"/>
+<part name="FID7" library="fiducials-jqi" deviceset="FIDUCIAL" device="-1.0MM"/>
+<part name="FID8" library="fiducials-jqi" deviceset="FIDUCIAL" device="-1.0MM"/>
 </parts>
 <sheets>
@@
 </plain>
 <instances>
-<instance part="X1" gate="G$1" x="35.56" y="67.31"/>
-<instance part="X2" gate="G$1" x="34.29" y="26.67"/>
+<instance part="X1" gate="G$1" x="35.56" y="67.31">
+<attribute name="PARTNO" x="35.56" y="67.31" size="1.778" layer="96" display="off"/>
+</instance>
+<instance part="X2" gate="G$1" x="34.29" y="26.67">
+<attribute name="PARTNO" x="34.29" y="26.67" size="1.778" layer="96" display="off"/>
+</instance>
 <instance part="FRAME1" gate="G$1" x="0" y="0"/>
 <instance part="FRAME1" gate="G$2" x="172.72" y="0"/>
@@
 <attribute name="PARTNO" x="52.07" y="29.21" size="1.778" layer="96" display="off"/>
 </instance>
+<instance part="FID1" gate="G$1" x="196.85" y="53.34"/>
+<instance part="FID2" gate="G$1" x="210.82" y="53.34"/>
+<instance part="FID3" gate="G$1" x="224.79" y="53.34"/>
+<instance part="FID4" gate="G$1" x="238.76" y="53.34"/>
+<instance part="FID5" gate="G$1" x="196.85" y="48.26"/>
+<instance part="FID6" gate="G$1" x="210.82" y="48.26"/>
+<instance part="FID7" gate="G$1" x="224.79" y="48.26"/>
+<instance part="FID8" gate="G$1" x="238.76" y="48.26"/>
 </instances>
 <busses>

Commit message: New 87Rb and 6Li antennas
I updated the eagle files with the new 87Rb and 6Li antenna designs from COMSOL.

DSB
Parts:
- removed C16: 3pF, jqi_passives:C_MLCC_SMDCMLCC_0402
- removed C17: 0.3pF, jqi_passives:C_MLCC_SMDCMLCC_0402
Connections:
- net COIL6LI_N: no longer C16.1, C16.2, C17.2
- net COIL6LI_P: no longer C17.1

Commit message: Updated values
Changed values in BOM to reflect results from prototype antennas.

DSB
Parts:
- C13, C14, C3, C4, C8, C9: PARTNO C3216X5R1H106K160AB -> CL31A106MBHNNNE
- RF: value 866 -> 220; PARTNO ERA-3AEB8660V -> TNPW0603220RBEEA
- RF1, RF2: value 866 -> 422; PARTNO ERA-3AEB8660V -> TNPW0603422RBEEA
- RG: value 95.3 -> 24.3; PARTNO ERA-2AEB95R3X -> RP73PF1E24R3BTD
- RG1, RG2: value 95.3 -> 46.4; PARTNO ERA-2AEB95R3X -> RP73PF1E46R4BTD
Changed lines of the file:
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@@
 </part>
 <part name="C3" library="jqi_passives" deviceset="C_MLCC_SMD" device="CMLCC_1206" value="10uF">
-<attribute name="PARTNO" value="C3216X5R1H106K160AB"/>
+<attribute name="PARTNO" value="CL31A106MBHNNNE"/>
 </part>
 <part name="C4" library="jqi_passives" deviceset="C_MLCC_SMD" device="CMLCC_1206" value="10uF">
-<attribute name="PARTNO" value="C3216X5R1H106K160AB"/>
+<attribute name="PARTNO" value="CL31A106MBHNNNE"/>
 </part>
 <part name="GND3" library="supply1" library_urn="urn:adsk.eagle:library:371" deviceset="GND" device=""/>
@@
 <attribute name="PARTNO" value="ERA-2AEB49R9X"/>
 </part>
-<part name="RG" library="jqi_passives" deviceset="R_SMD" device="R0402" value="95.3">
-<attribute name="PARTNO" value="ERA-2AEB95R3X"/>
+<part name="RG" library="jqi_passives" deviceset="R_SMD" device="R0402" value="24.3">
+<attribute name="PARTNO" value="RP73PF1E24R3BTD"/>
 </part>
-<part name="RF" library="jqi_passives" deviceset="R_SMD" device="R0603" value="866">
-<attribute name="PARTNO" value="ERA-3AEB8660V"/>
+<part name="RF" library="jqi_passives" deviceset="R_SMD" device="R0603" value="220">
+<attribute name="PARTNO" value="TNPW0603220RBEEA"/>
 </part>
 <part name="GND1" library="supply1" library_urn="urn:adsk.eagle:library:371" deviceset="GND" device=""/>
@@
 </part>
 <part name="C8" library="jqi_passives" deviceset="C_MLCC_SMD" device="CMLCC_1206" value="10uF">
-<attribute name="PARTNO" value="C3216X5R1H106K160AB"/>
+<attribute name="PARTNO" value="CL31A106MBHNNNE"/>
 </part>
 <part name="C9" library="jqi_passives" deviceset="C_MLCC_SMD" device="CMLCC_1206" value="10uF">
-<attribute name="PARTNO" value="C3216X5R1H106K160AB"/>
+<attribute name="PARTNO" value="CL31A106MBHNNNE"/>
 </part>
 <part name="GND8" library="supply1" library_urn="urn:adsk.eagle:library:371" deviceset="GND" device=""/>
@@
 <attribute name="PARTNO" value="ERA-2AEB49R9X"/>
 </part>
-<part name="RG1" library="jqi_passives" deviceset="R_SMD" device="R0402" value="95.3">
-<attribute name="PARTNO" value="ERA-2AEB95R3X"/>
+<part name="RG1" library="jqi_passives" deviceset="R_SMD" device="R0402" value="46.4">
+<attribute name="PARTNO" value="RP73PF1E46R4BTD"/>
 </part>
-<part name="RF1" library="jqi_passives" deviceset="R_SMD" device="R0603" value="866">
-<attribute name="PARTNO" value="ERA-3AEB8660V"/>
+<part name="RF1" library="jqi_passives" deviceset="R_SMD" device="R0603" value="422">
+<attribute name="PARTNO" value="TNPW0603422RBEEA"/>
 </part>
 <part name="GND9" library="supply1" library_urn="urn:adsk.eagle:library:371" deviceset="GND" device=""/>
@@
 </part>
 <part name="C13" library="jqi_passives" deviceset="C_MLCC_SMD" device="CMLCC_1206" value="10uF">
-<attribute name="PARTNO" value="C3216X5R1H106K160AB"/>
+<attribute name="PARTNO" value="CL31A106MBHNNNE"/>
 </part>
 <part name="C14" library="jqi_passives" deviceset="C_MLCC_SMD" device="CMLCC_1206" value="10uF">
-<attribute name="PARTNO" value="C3216X5R1H106K160AB"/>
+<attribute name="PARTNO" value="CL31A106MBHNNNE"/>
 </part>
 <part name="GND14" library="supply1" library_urn="urn:adsk.eagle:library:371" deviceset="GND" device=""/>
@@
 <attribute name="PARTNO" value="ERA-2AEB49R9X"/>
 </part>
-<part name="RG2" library="jqi_passives" deviceset="R_SMD" device="R0402" value="95.3">
-<attribute name="PARTNO" value="ERA-2AEB95R3X"/>
+<part name="RG2" library="jqi_passives" deviceset="R_SMD" device="R0402" value="46.4">
+<attribute name="PARTNO" value="RP73PF1E46R4BTD"/>
 </part>
-<part name="RF2" library="jqi_passives" deviceset="R_SMD" device="R0603" value="866">
-<attribute name="PARTNO" value="ERA-3AEB8660V"/>
+<part name="RF2" library="jqi_passives" deviceset="R_SMD" device="R0603" value="422">
+<attribute name="PARTNO" value="TNPW0603422RBEEA"/>
 </part>
 <part name="GND15" library="supply1" library_urn="urn:adsk.eagle:library:371" deviceset="GND" device=""/>
